File: CS42448_T4_TEST2.sch (KiCad schematic (older format))
At the start: 111 parts, among them J1 CUI_SJ1-3525N, J10 CUI_SJ1-3525N, J2 CUI_SJ1-3525N, J3 CUI_SJ1-3525N, J4 CUI_SJ1-3525N, J5 Conn_02x02_Top_Bottom, J6 Conn_02x07_Odd_Even, J7 CUI_SJ1-3525N, J8 CUI_SJ1-3525N, J9 CUI_SJ1-3525N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

Commit message: Added BOM in .csv format
The BOM contains sources for the components for Digikey, Mouser, and
PJRC
Parts:
- removed U4: Teensy4.0_28pin, project_libs:Teensy40_28pin, symbol CS42448_T4_TEST_symbols:Teensy4.0_28pin
- added U?: Teensy4.0_28pin, project_libs:Teensy40_28pin, symbol CS42448_T4_TEST_symbols:Teensy4.0_28pin

Commit message: Corrected 2x2 header pinout on schematic
Previously, the 2x2 header pinout on the schematic was top-bottom. That
has been changed to odd-even for consistency with the other header on
the schematic
Parts:
- J5: symbol Connector_Generic:Conn_02x02_Top_Bottom -> Connector_Generic:Conn_02x02_Odd_Even
- gave numbers to parts that had none: 1
Changed lines of the file:
@@
 	5000 6350 5400 6350
 $Comp
-L Connector_Generic:Conn_02x02_Top_Bottom J5
+L Connector_Generic:Conn_02x02_Odd_Even J5
 U 1 1 60CA2107
 P 7650 7000
@@
 $EndComp
 $Comp
-L CS42448_T4_TEST_symbols:Teensy4.0_28pin U?
+L CS42448_T4_TEST_symbols:Teensy4.0_28pin U4
 U 1 1 6048C8A8
 P 5500 1650
-F 0 "U?" H 5500 2517 50  0000 C CNN
+F 0 "U4" H 5500 2517 50  0000 C CNN
 F 1 "Teensy4.0_28pin" H 5500 2426 50  0000 C CNN
 F 2 "project_libs:Teensy40_28pin" H 5100 1100 50  0001 C CNN
